Commit message: Modification Haptic device driver application

File: 02-HapticDeviceDriver/kuka_iiwa.urdf (robot description, URDF)
Before this commit: robot kuka_iiwa, 8 links, 7 joints
Links:
- link link6: geometry visual box size=0.03 0.03 0.03; visual mesh filename=../../../Model/meshes_iiwa/link6.obj scale=1 1 1
