Commit message: Application Haptic guidances with Franka updated

File: 06-HapticGuidanceFranka/panda_arm.urdf (robot description, URDF)
Before this commit: robot panda, 8 links, 7 joints
Links:
- link link0: geometry visual mesh filename=../../../Model/meshes_panda/visual/link0.obj
- link link1: geometry visual mesh filename=../../../Model/meshes_panda/visual/link1.obj
- link link2: geometry visual mesh filename=../../../Model/meshes_panda/visual/link2.obj
- link link3: geometry visual mesh filename=../../../Model/meshes_panda/visual/link3.obj
- link link4: geometry visual mesh filename=../../../Model/meshes_panda/visual/link4.obj
- link link5: geometry visual mesh filename=../../../Model/meshes_panda/visual/link5.obj
- link link6: geometry visual mesh filename=../../../Model/meshes_panda/visual/link6.obj
- link link7: geometry collision sphere radius=0.04; visual mesh filename=../../../Model/meshes_panda/visual/link7.obj
