Commit message: Applications updated to last haptic controller, Added Connor's plane/line guidance, Application for Human-Robot interaction user study

File: 01-WorskpaceExtensionSimu/kuka_iiwa.urdf (robot description, URDF)
Before this commit: robot kuka_iiwa, 8 links, 7 joints
Links:
- link link6: geometry collision box size=0.03 0.03 0.03; visual box size=0.03 0.03 0.03

File: 04-HapticDeviceHumanInteraction/kuka_iiwa.urdf (robot description, URDF)
Before this commit: robot kuka_iiwa, 8 links, 7 joints
Links:
- link link6: geometry collision sphere radius=0.03; visual mesh filename=../../../Model/meshes_iiwa/link6.obj scale=1 1 1

Commit message: First demo of Haptic guidance and unified controller with Panda

File: 01-WorskpaceExtensionSimu/kuka_iiwa.urdf (robot description, URDF)
Before this commit: robot kuka_iiwa, 8 links, 7 joints
Links:
- link link6: geometry collision sphere radius=0.02; visual mesh filename=../../../Model/meshes_iiwa/link6.obj scale=1 1 1
