Commit message: Modification unified controller applications with contact normal to debug...

File: 10-UnifiedHapticControlCurvedSurfaceExperiment/panda_arm.urdf (robot description, URDF)
Before this commit: robot panda, 8 links, 7 joints
Links:
- link link7: geometry collision cylinder length=0.04 radius=0.015; visual cylinder length=0.04 radius=0.015

Commit message: unified haptic framework simulations

File: 10-UnifiedHapticControlCurvedSurfaceExperiment/panda_arm.urdf (robot description, URDF)
Before this commit: robot panda, 8 links, 7 joints
Links:
- link link7: geometry collision cylinder length=0.02 radius=0.015; visual cylinder length=0.02 radius=0.015
