Commit message: Test Kalman filter to estimate contact direction

File: 11-UnifiedHapticControlForceSpaceIdentification/panda_arm_sim.urdf (robot description, URDF)
Before this commit: robot panda, 8 links, 7 joints
Links:
- link link7: geometry collision sphere radius=0.02; visual cylinder length=0.047 radius=0.02
